Commit message: added structure and changed urdf joint names

File: leg_sim/simple_leg_pybullet/simple_leg_pybullet.urdf (robot description, URDF)
Before this commit: robot simple_leg_pybullet, 9 links, 8 joints
Links:
- removed link femur_servo1
- removed link femur_servo_arm1
- removed link leg_hip_servo_holder1
- removed link leg_knee_up1
- removed link shoulder_servo_arm1
- removed link tibia_servo1
- added link hip_servo_arm1, mass 0.0032701003729527518; collision mesh filename=meshes/hip_servo_arm1.stl scale=0.001 0.001 0.001; visual mesh filename=meshes/hip_servo_arm1.stl scale=0.001 0.001 0.001
- added link knee_servo1, mass 0.04604548230153534; collision mesh filename=meshes/knee_servo1.stl scale=0.001 0.001 0.001; visual mesh filename=meshes/knee_servo1.stl scale=0.001 0.001 0.001
- added link knee_servo_arm1, mass 0.0032701003729527518; collision mesh filename=meshes/knee_servo_arm1.stl scale=0.001 0.001 0.001; visual mesh filename=meshes/knee_servo_arm1.stl scale=0.001 0.001 0.001
- added link knee_servo_holder1, mass 0.03470303413377985; collision mesh filename=meshes/knee_servo_holder1.stl scale=0.001 0.001 0.001; visual mesh filename=meshes/knee_servo_holder1.stl scale=0.001 0.001 0.001
- added link leg_tibia1, mass 0.016745594670500637; collision mesh filename=meshes/leg_tibia1.stl scale=0.001 0.001 0.001; visual mesh filename=meshes/leg_tibia1.stl scale=0.001 0.001 0.001
Joints:
- removed joint Revolute_23
- removed joint Revolute_28
- removed joint Revolute_38
- removed joint Rigid_26
- added joint hip_joint: type continuous, parent base_link, child hip_servo_arm1, origin xyz=0.065722 0.013766 0.136395 rpy=0 0 0, axis -0.999994 0.0 0.003393
- added joint knee_joint: type continuous, parent knee_servo1, child knee_servo_arm1, origin xyz=-0.001385 -0.047866 -0.002762 rpy=0 0 0, axis 0.0 1.0 -0.0
- added joint tibia_joint: type continuous, parent leg_tibia1, child leg_ankle1, origin xyz=-0.049674 -0.013 -0.076733 rpy=0 0 0, axis 0.0 1.0 -0.0
- joint Rigid_24: child leg_hip_servo_holder1 -> knee_servo_holder1; parent shoulder_servo_arm1 -> hip_servo_arm1
- joint Rigid_25: child femur_servo1 -> knee_servo1; parent leg_hip_servo_holder1 -> knee_servo_holder1
- joint Rigid_37: child leg_knee_up1 -> leg_tibia1; parent femur_servo_arm1 -> knee_servo_arm1

Commit message: working simulation debug line & sin trajectory

File: leg_sim/simple_leg_pybullet/simple_leg_pybullet.urdf (robot description, URDF)
Before this commit: robot simple_leg_pybullet, 8 links, 7 joints
Links:
- added link tibia_servo1, mass 46.045481761973825; collision mesh filename=meshes/tibia_servo1.stl scale=0.001 0.001 0.001; visual mesh filename=meshes/tibia_servo1.stl scale=0.001 0.001 0.001
- link base_link: mass 0.04604548230153534 -> 46.04548176197378
- link hip_servo_arm1: mass 0.0032701003729527518 -> 3.2700935144949623
- link knee_servo1: mass 0.04604548230153534 -> 46.04548176197379
- link knee_servo_arm1: mass 0.0032701003729527518 -> 3.2700935144949637
- link knee_servo_holder1: mass 0.03470303413377985 -> 34.703034418237515
- link leg_ankle1: mass 0.022209898104400553 -> 22.20997101680633
- link leg_foot1Component161: mass 0.05068893861578388 -> 4.115954761083666
- link leg_tibia1: mass 0.016745594670500637 -> 16.745590583555348
Joints:
- added joint Rigid_26: type fixed, parent knee_servo_holder1, child tibia_servo1, origin xyz=0.589414 -0.044734 -0.070189 rpy=0 0 0
- joint Rigid_24: origin xyz=0.006 0.0 -2e-05 rpy=0 0 0 -> xyz=0.06 0.0 -0.000204 rpy=0 0 0
- joint Rigid_25: origin xyz=0.024622 0.029066 0.021604 rpy=0 0 0 -> xyz=0.101495 -0.044734 0.238129 rpy=0 0 0
- joint Rigid_35: origin xyz=0.073451 0.0066 -0.051929 rpy=0 0 0 -> xyz=0.734516 0.066 -0.519289 rpy=0 0 0
- joint Rigid_37: origin xyz=0.0 -0.006 0.0 rpy=0 0 0 -> xyz=0.0 -0.06 0.0 rpy=0 0 0
- joint hip_joint: origin xyz=0.065722 0.013766 0.136395 rpy=0 0 0 -> xyz=-0.505484 -0.128884 0.152548 rpy=0 0 0
- joint knee_joint: origin xyz=-0.001385 -0.047866 -0.002762 rpy=0 0 0 -> xyz=0.130875 -0.161266 -0.04971 rpy=0 0 0
- joint tibia_joint: origin xyz=-0.049674 -0.013 -0.076733 rpy=0 0 0 -> xyz=-0.496738 -0.13 -0.767329 rpy=0 0 0
