Commit message: haruki robot working

File: assets/haruki_urdf/quadrupedal.urdf (robot description, URDF)
Before this commit: robot quadrupedal_robot2, 13 links, 12 joints
Links:
- link base: geometry collision mesh filename=../assets/haruki_urdf/meshes/base.stl; visual mesh filename=../assets/haruki_urdf/meshes/base.stl
- link lf_abduction_link: geometry collision mesh filename=../assets/haruki_urdf/meshes/abduction_link.stl; visual mesh filename=../assets/haruki_urdf/meshes/abduction_link.stl
- link lf_lower_link: geometry collision mesh filename=../assets/haruki_urdf/meshes/lower_link.stl; visual mesh filename=../assets/haruki_urdf/meshes/lower_link.stl
- link lf_upper_link: geometry collision mesh filename=../assets/haruki_urdf/meshes/upper_link.stl; visual mesh filename=../assets/haruki_urdf/meshes/upper_link.stl
- link lh_abduction_link: geometry collision mesh filename=../assets/haruki_urdf/meshes/abduction_link.stl; visual mesh filename=../assets/haruki_urdf/meshes/abduction_link.stl
- link lh_lower_link: geometry collision mesh filename=../assets/haruki_urdf/meshes/lower_link.stl; visual mesh filename=../assets/haruki_urdf/meshes/lower_link.stl
- link lh_upper_link: geometry collision mesh filename=../assets/haruki_urdf/meshes/upper_link.stl; visual mesh filename=../assets/haruki_urdf/meshes/upper_link.stl
- link rf_abduction_link: geometry collision mesh filename=../assets/haruki_urdf/meshes/abduction_link.stl; visual mesh filename=../assets/haruki_urdf/meshes/abduction_link.stl
- link rf_lower_link: geometry collision mesh filename=../assets/haruki_urdf/meshes/lower_link.stl; visual mesh filename=../assets/haruki_urdf/meshes/lower_link.stl
- link rf_upper_link: geometry collision mesh filename=../assets/haruki_urdf/meshes/upper_link.stl; visual mesh filename=../assets/haruki_urdf/meshes/upper_link.stl
- link rh_abduction_link: geometry collision mesh filename=../assets/haruki_urdf/meshes/abduction_link.stl; visual mesh filename=../assets/haruki_urdf/meshes/abduction_link.stl
- link rh_lower_link: geometry collision mesh filename=../assets/haruki_urdf/meshes/lower_link.stl; visual mesh filename=../assets/haruki_urdf/meshes/lower_link.stl
- link rh_upper_link: geometry collision mesh filename=../assets/haruki_urdf/meshes/upper_link.stl; visual mesh filename=../assets/haruki_urdf/meshes/upper_link.stl
